File: hardware/klaviatar_pcb/keyboard.kicad_sch (KiCad schematic)
At the start: 88 parts, among them SW1 SA1, SW10 SA1, SW11 SA1, SW12 SA1, SW13 SA1, SW14 SA1, SW15 SA1, SW16 SA1, SW17 SA1, SW18 SA1, SW19 SA1, SW2 ESC, SW20 SA1, SW21 SA1, SW22 SA1, SW24 SA1, SW25 SA1, SW26 SA1, SW27 SA1, SW28 SA1, SW29 SA1, SW3 SA1, SW30 SA1, SW31 SA1, SW32 SA1, SW33 SA1, SW34 SA1, SW35 SA1, SW36 SA1, SW37 SA1, SW38 SA1, SW39 SA1, SW4 SA1, SW40 SA1, SW41 SA1, SW42 SA1, SW43 L, SW44 SA1, SW45 SA1, SW46 SA1, SW47 SA1, SW48 SA1, SW49 SA1, SW5 SA1, SW50 SA1, SW51 SA1, SW52 SA1, SW53 SA1, SW54 SA1, SW55 SA1, SW56 SA1, SW57 SA1, SW58 SA1, SW59 SA1, SW6 SA1, SW60 SA1, SW61 SA1, SW62 SA1, SW63 SA1, SW64 SA1, SW65 SA1, SW66 SA1, SW67 SA1, SW68 SA1, SW69 SA1, SW7 SA1, SW70 SA1, SW71 SA1, SW72 SA1, SW73 SA1, SW74 SA1, SW75 SA1, SW76 SA1, SW77 SA1, SW78 SA1, SW79 SA1, SW8 SA1, SW80 SA1, SW81 SA1, SW82 SA1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

Commit message: update sch
Parts:
- SW1: value SA1 -> "-"
Connections:
- net XT2_{9}: now also SW89.2; no longer SW89.1
- net XT1_{3}: now reaches SW14.2, SW27.2, SW28.2, SW3.2, SW53.2, SW54.2, SW55.2, SW56.2
- net XT1_{1}: now reaches SW1.2, SW12.2, SW24.2, SW45.2, SW46.2, SW47.2, SW48.2
- net XT1_{8}: now reaches SW19.2, SW37.2, SW38.2, SW73.2, SW74.2, SW75.2, SW76.2, SW8.2
- net XT1_{5}: now reaches SW16.2, SW31.2, SW32.2, SW5.2, SW61.2, SW62.2, SW63.2, SW64.2
- net XT1_{11}: now reaches SW11.2, SW22.2, SW43.2, SW44.2, SW85.2, SW86.2, SW87.2, SW88.2
- net XT1_{11}: no longer SW89.2
- net XT1_{6}: now reaches SW17.2, SW33.2, SW34.2, SW6.2, SW65.2, SW66.2, SW67.2, SW68.2
- net XT1_{10}: now reaches SW10.2, SW21.2, SW41.2, SW42.2, SW81.2, SW82.2, SW83.2, SW84.2
- net XT1_{2}: now reaches SW13.2, SW2.2, SW25.2, SW26.2, SW49.2, SW50.2, SW51.2, SW52.2
- net XT1_{7}: now reaches SW18.2, SW35.2, SW36.2, SW69.2, SW7.2, SW70.2, SW71.2, SW72.2
- net XT1_{4}: now reaches SW15.2, SW29.2, SW30.2, SW4.2, SW57.2, SW58.2, SW59.2, SW60.2
- net XT1_{9}: now reaches SW20.2, SW39.2, SW40.2, SW77.2, SW78.2, SW79.2, SW80.2, SW9.2
- new net XT1_{12}: SW89.1
Other:
- note added: "X, PORTD0..7+PORTC0..3"
- note added: "Y, PORTA0+PORTB0..7"
- moved on the sheet: SW89
Changed lines of the file:
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@@
   (junction (at 100.33 86.36) (diameter 0) (color 0 0 0 0)
   )
-  (junction (at 168.91 128.27) (diameter 0) (color 0 0 0 0)
-  )
   (junction (at 151.13 73.66) (diameter 0) (color 0 0 0 0)
   )
@@
     (stroke (width 0) (type default))
   )
-  (wire (pts (xy 168.91 128.27) (xy 168.91 148.59))
+  (wire (pts (xy 168.91 115.57) (xy 168.91 148.59))
     (stroke (width 0) (type default))
   )
@@
     (stroke (width 0) (type default))
   )
-  (wire (pts (xy 163.83 137.16) (xy 213.36 137.16))
-    (stroke (width 0) (type default))
-  )
   (wire (pts (xy 125.73 82.55) (xy 125.73 86.36))
     (stroke (width 0) (type default))
@@
     (stroke (width 0) (type default))
   )
+  (wire (pts (xy 176.53 135.89) (xy 176.53 148.59))
+    (stroke (width 0) (type default))
+  )
   (wire (pts (xy 151.13 73.66) (xy 163.83 73.66))
     (stroke (width 0) (type default))
@@
     (stroke (width 0) (type default))
   )
+  (wire (pts (xy 181.61 130.81) (xy 213.36 130.81))
+    (stroke (width 0) (type default))
+  )
   (wire (pts (xy 80.01 52.07) (xy 80.01 64.77))
     (stroke (width 0) (type default))
@@
     (stroke (width 0) (type default))
   )
-  (wire (pts (xy 163.83 133.35) (xy 163.83 137.16))
-    (stroke (width 0) (type default))
-  )
   (wire (pts (xy 130.81 115.57) (xy 130.81 148.59))
     (stroke (width 0) (type default))
@@
     (stroke (width 0) (type default))
   )
-  (wire (pts (xy 168.91 115.57) (xy 168.91 128.27))
-    (stroke (width 0) (type default))
-  )
   (wire (pts (xy 125.73 86.36) (xy 138.43 86.36))
     (stroke (width 0) (type default))
@@
     (stroke (width 0) (type default))
   )
+  (text "X, PORTD0..7+PORTC0..3" (at 85.09 162.56 0)
+    (effects (font (size 1.27 1.27)) (justify left bottom))
+  )
+  (text "Y, PORTA0+PORTB0..7" (at 223.52 77.47 0)
+    (effects (font (size 1.27 1.27)) (justify left bottom))
+  )
   (label "XT2_{1}" (at 196.85 35.56 0) (fields_autoplaced)
     (effects (font (size 1.27 1.27)) (justify left bottom))
@@
     (effects (font (size 1.27 1.27)) (justify left bottom))
   )
-  (label "XT2_{9}" (at 198.12 137.16 0) (fields_autoplaced)
+  (label "XT1_{10}" (at 156.21 138.43 90) (fields_autoplaced)
+    (effects (font (size 1.27 1.27)) (justify left bottom))
+  )
+  (label "XT1_{6}" (at 105.41 138.43 90) (fields_autoplaced)
+    (effects (font (size 1.27 1.27)) (justify left bottom))
+  )
+  (label "XT2_{9}" (at 196.85 130.81 0) (fields_autoplaced)
     (effects (font (size 1.27 1.27)) (justify left bottom))
   )
@@
     (effects (font (size 1.27 1.27)) (justify left bottom))
   )
+  (label "XT1_{4}" (at 80.01 138.43 90) (fields_autoplaced)
+    (effects (font (size 1.27 1.27)) (justify left bottom))
+  )
+  (label "XT1_{9}" (at 143.51 138.43 90) (fields_autoplaced)
+    (effects (font (size 1.27 1.27)) (justify left bottom))
+  )
   (label "XT2_{4}" (at 196.85 73.66 0) (fields_autoplaced)
     (effects (font (size 1.27 1.27)) (justify left bottom))
@@
     (effects (font (size 1.27 1.27)) (justify left bottom))
   )
+  (label "XT1_{12}" (at 176.53 144.78 90) (fields_autoplaced)
+    (effects (font (size 1.27 1.27)) (justify left bottom))
+  )
+  (label "XT1_{11}" (at 168.91 138.43 90) (fields_autoplaced)
+    (effects (font (size 1.27 1.27)) (justify left bottom))
+  )
   (label "XT2_{3}" (at 196.85 60.96 0) (fields_autoplaced)
     (effects (font (size 1.27 1.27)) (justify left bottom))
   )
+  (label "XT1_{1}" (at 41.91 138.43 90) (fields_autoplaced)
+    (effects (font (size 1.27 1.27)) (justify left bottom))
+  )
+  (label "XT1_{8}" (at 130.81 138.43 90) (fields_autoplaced)
+    (effects (font (size 1.27 1.27)) (justify left bottom))
+  )
+  (label "XT1_{5}" (at 92.71 138.43 90) (fields_autoplaced)
+    (effects (font (size 1.27 1.27)) (justify left bottom))
+  )
+  (label "XT1_{3}" (at 67.31 138.43 90) (fields_autoplaced)
+    (effects (font (size 1.27 1.27)) (justify left bottom))
+  )
+  (label "XT1_{7}" (at 118.11 138.43 90) (fields_autoplaced)
+    (effects (font (size 1.27 1.27)) (justify left bottom))
+  )
+  (label "XT1_{2}" (at 54.61 138.43 90) (fields_autoplaced)
+    (effects (font (size 1.27 1.27)) (justify left bottom))
+  )
   (symbol (lib_id "Switch:SW_Push_45deg") (at 64.77 92.71 90) (unit 1)
     (in_bom yes) (on_board yes) (dnp no)
@@
       (effects (font (size 1.27 1.27)) (justify right))
     )
-    (property "Value" "SA1" (at 31.75 30.48 90)
+    (property "Value" "\"-\"" (at 31.75 30.48 90)
       (effects (font (size 1.27 1.27)) (justify right))
     )
@@
     )
   )
-  (symbol (lib_id "Switch:SW_Push_45deg") (at 166.37 130.81 90) (unit 1)
-    (in_bom yes) (on_board yes) (dnp no)
-    (property "Reference" "SW89" (at 157.48 129.54 90)
-      (effects (font (size 1.27 1.27)) (justify right))
-    )
-    (property "Value" "F10" (at 157.48 132.08 90)
-      (effects (font (size 1.27 1.27)) (justify right))
-    )
-    (property "Footprint" "" (at 166.37 130.81 0)
-      (effects (font (size 1.27 1.27)) hide)
-    )
-    (property "Datasheet" "~" (at 166.37 130.81 0)
-      (effects (font (size 1.27 1.27)) hide)
-    )
+  (symbol (lib_id "Switch:SW_Push_45deg") (at 179.07 133.35 90) (unit 1)
+    (in_bom yes) (on_board yes) (dnp no)
+    (property "Reference" "SW89" (at 170.18 132.08 90)
+      (effects (font (size 1.27 1.27)) (justify right))
+    )
+    (property "Value" "F10" (at 170.18 134.62 90)
+      (effects (font (size 1.27 1.27)) (justify right))
+    )
+    (property "Footprint" "" (at 179.07 133.35 0)
+      (effects (font (size 1.27 1.27)) hide)
+    )
+    (property "Datasheet" "~" (at 179.07 133.35 0)
+      (effects (font (size 1.27 1.27)) hide)
+    )

Commit message: add custom pcb
Parts:
- SW1, SW10, SW11, SW14, SW15, SW16, SW17, SW18, SW19, SW2, SW20, SW21, SW22, SW26, SW27, SW28, SW29, SW3, SW30, SW31, SW32, SW33, SW34, SW35, SW36, SW37, SW38, SW39, SW4, SW40, SW41, SW42, SW43, SW44, SW46, SW47, SW48, SW49, SW5, SW50, SW51, SW52, SW53, SW54, SW55, SW56, SW57, SW58, SW59, SW6, SW60, SW61, SW62, SW63, SW64, SW65, SW66, SW67, SW68, SW69, SW7, SW70, SW71, SW72, SW73, SW74, SW75, SW76, SW77, SW78, SW79, SW8, SW80, SW81, SW82, SW83, SW84, SW85, SW86, SW87, SW88, SW89, SW9: footprint (none) -> Button_Switch_Keyboard:SW_Cherry_MX_1.00u_Plate
- SW12: value SA1 -> stop; footprint (none) -> Button_Switch_Keyboard:SW_Cherry_MX_1.00u_Plate
- SW13: value SA1 -> Tab; footprint (none) -> Button_Switch_Keyboard:SW_Cherry_MX_1.00u_Plate
- SW24: value SA1 -> lshift; footprint (none) -> Button_Switch_Keyboard:SW_Cherry_MX_1.00u_Plate
- SW25: value SA1 -> caps; footprint (none) -> Button_Switch_Keyboard:SW_Cherry_MX_1.00u_Plate
- SW45: value SA1 -> rshift; footprint (none) -> Button_Switch_Keyboard:SW_Cherry_MX_1.00u_Plate
Connections:
- net XT2_{4}: no longer SW24.1
- net XT2_{5}: now also SW24.1
