File: hardware/klaviatar_pcb/klaviatar_pcb.kicad_sch (KiCad schematic)
At the start: 2 parts, among them J2 keyboard_out, J3 keyboard_in

Commit message: keyboard pcb
Parts:
- removed J3: keyboard_in, symbol Connector:Conn_01x09_Socket
- added J1: Conn_01x12_Socket, symbol Connector:Conn_01x12_Socket
- added U1: PIC18F4550-IP, Package_DIP:DIP-40_W15.24mm, symbol MCU_Microchip_PIC18:PIC18F4550-IP
- added Y1: Crystal, symbol Device:Crystal
Connections:
- net X1: now reaches J2.1 (Pin_1)
- net X1: now also U1.33 (RB0/AN12/INT0/FLT0/SDI/SDA)
- net X2: now reaches J2.2 (Pin_2)
- net X2: now also U1.34 (RB1/AN10/INT1/SCK/SCL)
- net X3: now reaches J2.3 (Pin_3)
- net X3: now also U1.35 (RB2/AN8/INT2/VMO)
- net X4: now reaches J2.4 (Pin_4)
- net X4: now also U1.36 (RB3/AN9/CCP2/VPO)
- net X5: now reaches J2.5 (Pin_5)
- net X5: now also U1.37 (RB4/AN11/KBI0/CSSPP)
- net X6: now reaches J2.6 (Pin_6)
- net X6: now also U1.38 (RB5/KBI1/PGM)
- net X7: now reaches J2.7 (Pin_7)
- net X7: now also U1.39 (RB6/KBI2/PGC)
- net X8: now reaches J2.8 (Pin_8)
- net X8: now also U1.40 (RB7/KBI3/PGD)
- net X9: now reaches J2.9 (Pin_9)
- new net: U1.11 (VDD), U1.32 (VDD)
- new net: U1.13 (OSC1/CLKI), Y1.1
- new net: U1.14 (RA6/OSC2/CLKO), Y1.2
- new net GND: U1.12 (VSS), U1.31 (VSS)
- new net Y1: J1.1 (Pin_1)
- new net Y10: J1.10 (Pin_10)
- new net Y11: J1.11 (Pin_11)
- new net Y12: J1.12 (Pin_12)
- new net Y2: J1.2 (Pin_2)
- new net Y3: J1.3 (Pin_3)
- new net Y4: J1.4 (Pin_4)
- new net Y5: J1.5 (Pin_5)
- new net Y6: J1.6 (Pin_6)
- new net Y7: J1.7 (Pin_7)
- new net Y8: J1.8 (Pin_8)
- new net Y9: J1.9 (Pin_9)
Other:
- added sheet keyboard (keyboard.kicad_sch)
- moved on the sheet: J2

Commit message: add connections
Parts:
- added D1, D10, D11, D12, D2, D3, D4, D5, D6, D7, D8, D9: 1N4148, Diode_THT:D_DO-35_SOD27_P7.62mm_Horizontal, symbol Diode:1N4148
- added R1, R10, R11, R12, R13, R14, R15, R16, R17, R18, R19, R2, R20, R21, R3, R4, R5, R6, R7, R8, R9: R, symbol Device:R
Connections:
- net X9 is gone; now on an unnamed net: J2.9 (Pin_9)
- net at U1.1 (Vpp/~{MCLR}/RE3): now also R12.2
- net at U1.10 (OESPP/AN7/RE2): now also R11.2
- net at U1.19 (SPP0/RD0): now also R1.2
- net at U1.2 (RA0/AN0): now also R21.2
- net at U1.20 (SPP1/RD1): now also R2.2
- net at U1.21 (SPP2/RD2): now also R3.2
- net at U1.22 (SPP3/RD3): now also R4.2
- net at U1.27 (SPP4/RD4): now also R5.2
- net at U1.28 (P1B/SPP5/RD5): now also R6.2
- net at U1.29 (P1C/SPP6/RD6): now also R7.2
- net at U1.30 (P1D/SPP7/RD7): now also R8.2
- net at U1.8 (CK1SPP/AN5/RE0): now also R9.2
- net at U1.9 (CK2SPP/AN6/RE1): now also R10.2
- net X1: no longer names the net of J2.1 (Pin_1), U1.33 (RB0/AN12/INT0/FLT0/SDI/SDA)
- net X1: now also R14.2
- net X2: no longer names the net of J2.2 (Pin_2), U1.34 (RB1/AN10/INT1/SCK/SCL)
- net X2: now also R15.2
- net X3: no longer names the net of J2.3 (Pin_3), U1.35 (RB2/AN8/INT2/VMO)
- net X3: now also R16.2
- net X4: no longer names the net of J2.4 (Pin_4), U1.36 (RB3/AN9/CCP2/VPO)
- net X4: now also R17.2
- net X5: no longer names the net of J2.5 (Pin_5), U1.37 (RB4/AN11/KBI0/CSSPP)
- net X5: now also R13.2
- net X6: no longer names the net of J2.6 (Pin_6), U1.38 (RB5/KBI1/PGM)
- net X6: now also R18.2
- net X7: no longer names the net of J2.7 (Pin_7), U1.39 (RB6/KBI2/PGC)
- net X7: now also R19.2
- net X8: no longer names the net of J2.8 (Pin_8), U1.40 (RB7/KBI3/PGD)
- net X8: now also R20.2
- net Y1: no longer names the net of J1.1 (Pin_1)
- net Y1: now also D1.2 (A)
- net Y10: no longer names the net of J1.10 (Pin_10)
- net Y10: now also D10.2 (A)
- net Y11: no longer names the net of J1.11 (Pin_11)
- net Y11: now also D11.2 (A)
- net Y12: no longer names the net of J1.12 (Pin_12)
- net Y12: now also D12.2 (A)
- net Y2: no longer names the net of J1.2 (Pin_2)
- net Y2: now also D2.2 (A)
- net Y3: no longer names the net of J1.3 (Pin_3)
- net Y3: now also D3.2 (A)
- net Y4: no longer names the net of J1.4 (Pin_4)
- net Y4: now also D4.2 (A)
- net Y5: no longer names the net of J1.5 (Pin_5)
- net Y5: now also D5.2 (A)
- net Y6: no longer names the net of J1.6 (Pin_6)
- net Y6: now also D6.2 (A)
- net Y7: no longer names the net of J1.7 (Pin_7)
- net Y7: now also D7.2 (A)
- net Y8: no longer names the net of J1.8 (Pin_8)
- net Y8: now also D8.2 (A)
- net Y9: no longer names the net of J1.9 (Pin_9)
- net Y9: now also D9.2 (A)
- new net: D1.1 (K), R1.1
- new net: R13.1, R14.1, R15.1, R16.1, R17.1, R18.1, R19.1, R20.1, R21.1
- new net: D8.1 (K), R8.1
- new net: D4.1 (K), R4.1
- new net: D2.1 (K), R2.1
- new net: D12.1 (K), R12.1
- new net: D5.1 (K), R5.1
- new net: D7.1 (K), R7.1
- new net: D6.1 (K), R6.1
- new net: D10.1 (K), R10.1
- new net: D9.1 (K), R9.1
- new net: D3.1 (K), R3.1
- new net: D11.1 (K), R11.1
Other:
- removed sheet keyboard
- moved on the sheet: J1, J2, U1, Y1

Commit message: add custom pcb
Other:
- added sheet Keyboard (keyboard.kicad_sch)
Changed lines of the file:
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@@
+    )
+  )
+  (sheet (at 203.2 31.75) (size 49.53 20.32) (fields_autoplaced)
+    (stroke (width 0.1524) (type solid))
+    (fill (color 0 0 0 0.0000))
+    (property "Sheetname" "Keyboard" (at 203.2 31.0384 0)
+      (effects (font (size 1.27 1.27)) (justify left bottom))
+    )
+    (property "Sheetfile" "keyboard.kicad_sch" (at 203.2 52.6546 0)
+      (effects (font (size 1.27 1.27)) (justify left top))
+    )
+    (instances
+      (project "klaviatar_pcb"
+        (path "/dac1fbdd-4b4f-4871-b040-711665a635b2" (page "2"))
+      )
     )
   )
